File: KiCad/subtone.kicad_pcb (KiCad board)
At the start: 2 copper layers, 52.1 x 35.6 mm, 14 parts, among them J1 7P Header, J2 Conn_01x07_Pin, J3 3P Header, SW1 Encoder, U1 MODULE-XIAO-RP2040

Commit message: * Added screenshot * Default to 5V on J3 Header
Connections:
- JP1 pad 1: +3V3 -> +5V
- JP1 pad 3: +5V -> +3V3
Changed lines of the file:
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@@
       (stroke (width 0.05) (type solid)) (layer "F.CrtYd"))
     (pad "1" smd rect (at -1.3 0 270) (size 1 1.5) (layers "F.Cu" "F.Mask")
-      (net 2 "+3V3") (pinfunction "A") (pintype "passive"))
+      (net 12 "+5V") (pinfunction "A") (pintype "passive"))
     (pad "2" smd rect (at 0 0 270) (size 1 1.5) (layers "F.Cu" "F.Mask")
       (net 17 "Net-(J3-Pin_2)") (pinfunction "C") (pintype "passive"))
     (pad "3" smd rect (at 1.3 0 270) (size 1 1.5) (layers "F.Cu" "F.Mask")
-      (net 12 "+5V") (pinfunction "B") (pintype "passive"))
+      (net 2 "+3V3") (pinfunction "B") (pintype "passive"))
   )
   (footprint "Connector_PinHeader_2.54mm:PinHeader_1x07_P2.54mm_Vertical" (layer "F.Cu")
